Commit message: 将dae模型文件以绝对路径写入urdf以导入到rviz2，但模型文件有问题；添加了可操作度计算

File: model/franka_panda_urdf/robots/panda_arm_tau.urdf (robot description, URDF)
Before this commit: robot panda, 10 links, 9 joints
Links:
- link link0: geometry collision mesh filename=file:///home/cyh/panda_ros2/model/franka_panda_urdf/meshes/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; visual mesh filename=file:///home/cyh/panda_ros2/model/franka_panda_urdf/meshes/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
- link link1: geometry collision mesh filename=file:///home/cyh/panda_ros2/model/franka_panda_urdf/meshes/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; visual mesh filename=file:///home/cyh/panda_ros2/model/franka_panda_urdf/meshes/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
- link link2: geometry collision mesh filename=file:///home/cyh/panda_ros2/model/franka_panda_urdf/meshes/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; visual mesh filename=file:///home/cyh/panda_ros2/model/franka_panda_urdf/meshes/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
- link link3: geometry collision mesh filename=file:///home/cyh/panda_ros2/model/franka_panda_urdf/meshes/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; visual mesh filename=file:///home/cyh/panda_ros2/model/franka_panda_urdf/meshes/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
- link link4: geometry collision mesh filename=file:///home/cyh/panda_ros2/model/franka_panda_urdf/meshes/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; visual mesh filename=file:///home/cyh/panda_ros2/model/franka_panda_urdf/meshes/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
- link link5: geometry collision mesh filename=file:///home/cyh/panda_ros2/model/franka_panda_urdf/meshes/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; visual mesh filename=file:///home/cyh/panda_ros2/model/franka_panda_urdf/meshes/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
- link link6: geometry collision mesh filename=file:///home/cyh/panda_ros2/model/franka_panda_urdf/meshes/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; visual mesh filename=file:///home/cyh/panda_ros2/model/franka_panda_urdf/meshes/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
- link link7: geometry collision mesh filename=file:///home/cyh/panda_ros2/model/franka_panda_urdf/meshes/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; visual mesh filename=file:///home/cyh/panda_ros2/model/franka_panda_urdf/meshes/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

File: src/panda_ros/model/panda_tau_sim.urdf (robot description, URDF)
Before this commit: robot panda, 10 links, 9 joints
Links:
- link link0: geometry collision mesh filename=file:///home/cyh/panda_ros2/model/franka_panda_urdf/meshes/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; visual mesh filename=file:///home/cyh/panda_ros2/model/franka_panda_urdf/meshes/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
- link link1: geometry collision mesh filename=file:///home/cyh/panda_ros2/model/franka_panda_urdf/meshes/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; visual mesh filename=file:///home/cyh/panda_ros2/model/franka_panda_urdf/meshes/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
- link link2: geometry collision mesh filename=file:///home/cyh/panda_ros2/model/franka_panda_urdf/meshes/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; visual mesh filename=file:///home/cyh/panda_ros2/model/franka_panda_urdf/meshes/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
- link link3: geometry collision mesh filename=file:///home/cyh/panda_ros2/model/franka_panda_urdf/meshes/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; visual mesh filename=file:///home/cyh/panda_ros2/model/franka_panda_urdf/meshes/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
- link link4: geometry collision mesh filename=file:///home/cyh/panda_ros2/model/franka_panda_urdf/meshes/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; visual mesh filename=file:///home/cyh/panda_ros2/model/franka_panda_urdf/meshes/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
- link link5: geometry collision mesh filename=file:///home/cyh/panda_ros2/model/franka_panda_urdf/meshes/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; visual mesh filename=file:///home/cyh/panda_ros2/model/franka_panda_urdf/meshes/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
- link link6: geometry collision mesh filename=file:///home/cyh/panda_ros2/model/franka_panda_urdf/meshes/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; visual mesh filename=file:///home/cyh/panda_ros2/model/franka_panda_urdf/meshes/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
- link link7: geometry collision mesh filename=file:///home/cyh/panda_ros2/model/franka_panda_urdf/meshes/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; visual mesh filename=file:///home/cyh/panda_ros2/model/franka_panda_urdf/meshes/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
