Commit message: 避障NMPC小demo,相对比较稳定

File: src/panda_ros/model/panda_tau_sim.urdf (robot description, URDF)
Before this commit: robot panda, 10 links, 9 joints
Links:
- link hand: geometry visual sphere radius=0.060; visual sphere radius=0.060
- link link3: geometry collision mesh filename=file:///home/cyh/panda_ros2/model/franka_panda_urdf/meshes/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; visual mesh filename=file:///home/cyh/panda_ros2/model/franka_panda_urdf/meshes/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
- link link4: geometry collision mesh filename=file:///home/cyh/panda_ros2/model/franka_panda_urdf/meshes/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; visual mesh filename=file:///home/cyh/panda_ros2/model/franka_panda_urdf/meshes/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
- link link5: geometry collision mesh filename=file:///home/cyh/panda_ros2/model/franka_panda_urdf/meshes/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; visual mesh filename=file:///home/cyh/panda_ros2/model/franka_panda_urdf/meshes/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
- link link6: geometry collision mesh filename=file:///home/cyh/panda_ros2/model/franka_panda_urdf/meshes/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; visual mesh filename=file:///home/cyh/panda_ros2/model/franka_panda_urdf/meshes/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
- link link7: geometry collision mesh filename=file:///home/cyh/panda_ros2/model/franka_panda_urdf/meshes/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; visual mesh filename=file:///home/cyh/panda_ros2/model/franka_panda_urdf/meshes/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
